File: Constant Current Driver.kicad_sch (KiCad schematic)
At the start: 5 parts, among them Q1 NPN, Q2 NPN

Commit message: Constant Current Driver Revision 1
Parts:
- removed Q1, Q2: NPN, symbol Simulation_SPICE:NPN
- removed R2: R_Shunt, symbol Device:R_Shunt
- added C1, C2: C, symbol Device:C
- added D2, D3, D4, D5, D6: LED, symbol Device:LED
- added Q1, Q2, Q3: RS9N50D, Package_TO_SOT_SMD:TO-252-2, symbol Transistor_FET:RS9N50D
- added R10, R11, R12, R3, R4, R5, R7, R8: R, symbol Device:R
- added R2, R6, R9: R SHUNT, symbol Device:R
- added U1: Nucleo_L432KC, symbol nucleo_stm32:Nucleo_L432KC
- added U10: LP38691SD-2.5, Package_SON:WSON-6-1EP_3x3mm_P0.95mm, symbol Regulator_Linear:LP38691SD-2.5
- added U2, U5, U8: TLV172IDCK, Package_TO_SOT_SMD:SOT-353_SC-70-5, symbol Amplifier_Operational:TLV172IDCK
- added U3, U4, U7: NSL-32, OptoDevice:Luna_NSL-32, symbol Isolator:NSL-32
Connections:
- net GND: now also R2.2, R6.2, R9.2, U2.1 (+), U5.1 (+), U8.1 (+)
- net at R1.2: now also Q1.2 (D)
- net at D1.1 (K): now also R2.1, U2.3 (-)
- net VCC: no longer names the net of D1.2 (A)
- net VCC: now also D2.1 (K); no longer R1.1
- new net: D4.1 (K), R6.1, U5.3 (-)
- new net: D3.1 (K), D4.2 (A)
- new net: R4.1, U4.3 (R), U4.4 (R)
- new net: Q2.1 (G), R4.2
- new net: D6.1 (K), R9.1, U8.3 (-)
- new net: D5.1 (K), D6.2 (A)
- new net: R12.2, U7.1 (A)
- new net: D3.2 (A), Q2.3 (S)
- new net: R7.1, U7.3 (R), U7.4 (R)
- new net: Q3.1 (G), R7.2
- new net: Q3.2 (D), R8.2
- new net: D5.2 (A), Q3.3 (S)
- new net: R11.2, U4.1 (A)
- new net: D2.2 (A), Q1.3 (S)
- new net: Q2.2 (D), R5.2
- new net: Q1.1 (G), R3.2
- new net: R3.1, U3.3 (R), U3.4 (R)
- new net: R10.2, U3.1 (A)
- new net ADC1_IN5: U1.19 (A0), U2.4, U5.4, U8.4
- new net FT_a: C1.2, U1.20 (A1), U10.1 (IN), U10.6 (IN)
- new net GND1: C1.1, C2.2, U1.29 (GND), U10.2 (GND), U10.7 (EP), U3.2 (K), U4.2 (K), U7.2 (K)
- new net VDD1: R1.1
- new net VDD2: R5.1
- new net VDD3: R8.1
- new net Vout: C2.1, R10.1, R11.1, R12.1, U10.4 (OUT), U10.5 (SNS)
- no-connect marks 0 -> 33
Other:
- moved on the sheet: D1, R1

Commit message: finished schematic!
Connections:
- net GND: now also C1.1, C2.2, U1.29 (GND), U10.2 (GND), U10.7 (EP), U2.2 (V-), U2.3 (-), U5.5 (V+), U8.5 (V+); no longer U2.1 (+)
- net GND1: no longer C1.1, C2.2, U1.29 (GND), U10.2 (GND), U10.7 (EP)
- net at D1.1 (K), R2.1: now also U2.1 (+); no longer U2.3 (-)
- net +3.3V: now reaches U1.17 (+3V3)
- net +3.3V: now also U2.5 (V+), U5.2 (V-), U8.2 (V-)
- net PA_2: now reaches U1.21 (A2)
- net PA_2: now also U2.4
- net PA_3: now reaches U1.22 (A3)
- net PA_3: now also U5.4
- net ADC1_IN5 renamed PA_0
- net PA_0: no longer U2.4, U5.4
- net FT_a renamed PA_1
- no-connect marks 33 -> 24
Other:
- moved on the sheet: U2

Commit message: Heliosphere v1.2
Parts:
- removed C1, C2: C, symbol Device:C
- removed D1, D2, D3, D4, D5, D6: LED, symbol Device:LED
- removed Q1, Q2, Q3: RS9N50D, Package_TO_SOT_SMD:TO-252-2, symbol Transistor_FET:RS9N50D
- removed R1, R10, R11, R12, R3, R4, R5, R7, R8: R, symbol Device:R
- removed R2, R6, R9: R SHUNT, symbol Device:R
- removed U1: Nucleo_L432KC, symbol nucleo_stm32:Nucleo_L432KC
- removed U10: LP38691SD-2.5, Package_SON:WSON-6-1EP_3x3mm_P0.95mm, symbol Regulator_Linear:LP38691SD-2.5
- removed U2, U5, U8: TLV172IDCK, Package_TO_SOT_SMD:SOT-353_SC-70-5, symbol Amplifier_Operational:TLV172IDCK
- removed U3, U4, U7: NSL-32, OptoDevice:Luna_NSL-32, symbol Isolator:NSL-32
Connections:
- no-connect marks 24 -> 0
Other:
- added sheet LED Board 1 (ConstantCurrentLED1.kicad_sch)
- added sheet LED Board 2 (CurrentDriverLED2.kicad_sch)
- added sheet LED Board 3 (CurrentDriverLED3.kicad_sch)
- added sheet MCU (CurrentDriverMCU.kicad_sch)
- note added: "Constant Current Driver v1.2"
