File: MCU/RTDControls.kicad_sch (KiCad schematic)
At the start: 2 parts, among them U10 AMC1301DWVR

Commit message: Finalized schematic and started layout
Parts:
- removed C9: 10nF, Capacitor_SMD:C_1206_3216Metric, symbol Device:C
- removed U10: AMC1301DWVR, AMC1301DWVR:SOIC127P1150X280-8N, symbol AMC1301:AMC1301DWVR
- added R14: 10k, Resistor_SMD:R_0603_1608Metric_Pad0.98x0.95mm_HandSolder, symbol Device:R
- added U9: INA333xxDGK, Package_SO:VSSOP-8_3x3mm_P0.65mm, symbol Amplifier_Instrumentation:INA333xxDGK
Connections:
- net GND: now also U9.2 (-), U9.4 (V-), U9.5 (Ref)
- net PA0: now also U9.6
- net RTD: now also U9.3 (+)
- new net: R14.1, U9.1 (Rg)
- new net: R14.2, U9.8 (Rg)
- new net +5V: U9.7 (V+)
Other:
- note added: "5 -- VOUTN -- PB0 6 -- VOUTP -- PA0"
- note added: "G = 2 = 1+ (100k/100k) VOUT_MAX = (5/(160+300)) * 160 * 2 = 3.3 I_MIN = 10.87 mA VOUT_MIN = (5/(400)) * 100 * 2 = 2.5 I_MAX = 12.5 mA"
- note added: "isolation is no longer needed"
- note removed: "VINN measures one side of the RTD VINP measures the other side of the RTD (GND1)"

Commit message: Adjusted trace widths. Added ferrite beads. Changed connectors to fit new trace widths. Added +3V3 fill zone in B.Cu. Fixed silkscreen placements.
Other:
- note added: "G = 2 = 1+ (100k/100k) RTD Resistance @ 155 C = 159.19 RTD Resistance @ 20 C = 107.79 VOUT_MAX = (5/(159.19+360)) * 159.19 * 2 = 3.066 V I_MIN = 9.63 mA @ 155 C VOUT_MIN = (5/(107.79+360)) * 107.79 * 2 = 2.304 V I_MAX = 10.69 mA @ 20 C"
- note removed: "G = 2 = 1+ (100k/100k) VOUT_MAX = (5/(160+300)) * 160 * 2 = 3.3 I_MIN = 10.87 mA VOUT_MIN = (5/(400)) * 100 * 2 = 2.5 I_MAX = 12.5 mA"
- note removed: "isolation is no longer needed"
Changed lines of the file:
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@@
 		)
 	)
-	(text "isolation is no longer needed\n"
+	(text "G = 2 = 1+ (100k/100k)\nRTD Resistance @ 155 C = 159.19\nRTD Resistance @ 20 C = 107.79\n\nVOUT_MAX = (5/(159.19+360)) * 159.19 * 2 = 3.066 V\nI_MIN = 9.63 mA @ 155 C\nVOUT_MIN = (5/(107.79+360)) * 107.79 * 2 = 2.304 V\nI_MAX = 10.69 mA @ 20 C"
 		(exclude_from_sim no)
-		(at 150.368 130.302 0)
+		(at 143.51 117.094 0)
 		(effects
 			(font
-				(size 1.27 1.27)
-			)
-		)
-	)
-	(text "G = 2 = 1+ (100k/100k)\n\nVOUT_MAX = (5/(160+300)) * 160 * 2 = 3.3\nI_MIN = 10.87 mA\nVOUT_MIN = (5/(400)) * 100 * 2 = 2.5\nI_MAX = 12.5 mA"
-		(exclude_from_sim no)
-		(at 139.446 113.538 0)
-		(effects
-			(font
