File: MCU/_autosave-LED.CONTROLS1.kicad_sch (KiCad schematic)
At the start: 21 parts, among them U3 HHG1D-1, U4 AMC3302QDWERQ1

Commit message: increased footprint sizes
Parts:
- C9: footprint Capacitor_SMD:C_0201_0603Metric_Pad0.64x0.40mm_HandSolder -> Capacitor_SMD:C_0603_1608Metric_Pad1.08x0.95mm_HandSolder
Changed lines of the file:
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@@
 			)
 		)
-		(property "Footprint" "Capacitor_SMD:C_0201_0603Metric_Pad0.64x0.40mm_HandSolder"
+		(property "Footprint" "Capacitor_SMD:C_0603_1608Metric_Pad1.08x0.95mm_HandSolder"
 			(at 213.0552 86.36 0)
 			(effects
@@
 			)
 		)
-		(property "Datasheet" "https://search.murata.co.jp/Ceramy/image/img/A01X/G101/ENG/GRM033C71C104KE14-01.pdf"
+		(property "Datasheet" "https://www.mouser.com/datasheet/3/72/1/KEM_C1002_X7R_SMD.pdf"
 			(at 212.09 82.55 0)
 			(effects
@@
 			)
 		)
-		(property "Description" "0.1 µF ±10% 16V Ceramic Capacitor X7S 0201 (0603 Metric)"
+		(property "Description" "Multilayer Ceramic Capacitors MLCC - SMD/SMT 50V 0.1uF X7R 0603 10%"
 			(at 212.09 82.55 0)
 			(effects
