File: MCU/RTD.kicad_sch (KiCad schematic)
At the start: 9 parts

Commit message: final?
Parts:
- gave numbers to parts that had none: 1
Connections:
- net D3 renamed CS
- net D7 renamed DRDY
- removed net DIAG: R15.2, R16.2, R17.2, R18.2
- net PA5 renamed SCLK
- net PA6 renamed SDO
- net PA7 renamed SDI
- new net FORCE+: R15.2
- new net FORCE-: R18.2
- new net RTDIN+: R16.2
- new net RTDIN-: R17.2
Changed lines of the file:
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@@
+	(wire
+		(pts
+			(xy 96.52 92.71) (xy 99.06 92.71)
+		)
+		(stroke
+			(width 0)
+			(type default)
+		)
+	)
 	(wire
 		(pts
@@
 	(wire
 		(pts
+			(xy 96.52 102.87) (xy 99.06 102.87)
+		)
+		(stroke
+			(width 0)
+			(type default)
+		)
+	)
+	(wire
+		(pts
 			(xy 148.59 114.3) (xy 154.94 114.3)
 		)
@@
 	(wire
 		(pts
+			(xy 96.52 95.25) (xy 99.06 95.25)
+		)
+		(stroke
+			(width 0)
+			(type default)
+		)
+	)
+	(wire
+		(pts
+			(xy 96.52 97.79) (xy 99.06 97.79)
+		)
+		(stroke
+			(width 0)
+			(type default)
+		)
+	)
+	(wire
+		(pts
 			(xy 135.89 109.22) (xy 135.89 110.49)
 		)
@@
 	(wire
 		(pts
-			(xy 97.79 95.25) (xy 99.06 95.25)
-		)
-		(stroke
-			(width 0)
-			(type default)
-		)
-	)
-	(wire
-		(pts
 			(xy 148.59 111.76) (xy 154.94 111.76)
 		)
@@
 	(wire
 		(pts
-			(xy 97.79 102.87) (xy 99.06 102.87)
-		)
-		(stroke
-			(width 0)
-			(type default)
-		)
-	)
-	(wire
-		(pts
 			(xy 151.13 120.65) (xy 151.13 116.84)
 		)
@@
 	(wire
 		(pts
-			(xy 97.79 92.71) (xy 99.06 92.71)
-		)
-		(stroke
-			(width 0)
-			(type default)
-		)
-	)
-	(wire
-		(pts
 			(xy 144.78 120.65) (xy 151.13 120.65)
 		)
@@
 	(wire
 		(pts
+			(xy 96.52 100.33) (xy 99.06 100.33)
+		)
+		(stroke
+			(width 0)
+			(type default)
+		)
+	)
+	(wire
+		(pts
 			(xy 133.35 109.22) (xy 133.35 113.03)
 		)
@@
 	(wire
 		(pts
-			(xy 97.79 97.79) (xy 99.06 97.79)
-		)
-		(stroke
-			(width 0)
-			(type default)
-		)
-	)
-	(wire
-		(pts
 			(xy 116.84 74.93) (xy 116.84 87.63)
 		)
@@
 	(wire
 		(pts
-			(xy 97.79 100.33) (xy 99.06 100.33)
-		)
-		(stroke
-			(width 0)
-			(type default)
-		)
-	)
-	(wire
-		(pts
 			(xy 132.08 100.33) (xy 132.08 102.87)
 		)
@@
 		)
 	)
-	(label "PA7"
-		(at 97.79 95.25 180)
-		(effects
-			(font
-				(size 1.27 1.27)
-			)
-			(justify right bottom)
-		)
-	)
-	(label "D3"
-		(at 97.79 100.33 180)
-		(effects
-			(font
-				(size 1.27 1.27)
-			)
-			(justify right bottom)
-		)
-	)
-	(label "D7"
-		(at 97.79 92.71 180)
-		(effects
-			(font
-				(size 1.27 1.27)
-			)
-			(justify right bottom)
-		)
-	)
-	(label "PA6"
-		(at 97.79 102.87 180)
-		(effects
-			(font
-				(size 1.27 1.27)
-			)
-			(justify right bottom)
-		)
-	)
-	(label "PA5"
-		(at 97.79 97.79 180)
-		(effects
-			(font
-				(size 1.27 1.27)
-			)
-			(justify right bottom)
-		)
-	)
-	(hierarchical_label "DIAG"
+	(hierarchical_label "RTDIN-"
 		(shape input)
 		(at 154.94 114.3 0)
@@
 		)
 	)
-	(hierarchical_label "DIAG"
+	(hierarchical_label "SDI"
+		(shape input)
+		(at 96.52 95.25 180)
+		(effects
+			(font
+				(size 1.27 1.27)
+			)
+			(justify right)
+		)
+	)
+	(hierarchical_label "FORCE-"
 		(shape input)
 		(at 154.94 116.84 0)
@@
 		)
 	)
-	(hierarchical_label "DIAG"
+	(hierarchical_label "FORCE+"
 		(shape input)
 		(at 154.94 109.22 0)
@@
 		)
 	)
-	(hierarchical_label "DIAG"
+	(hierarchical_label "RTDIN+"
 		(shape input)
 		(at 154.94 111.76 0)
@@
 			)
 			(justify left)
+		)
+	)
+	(hierarchical_label "SDO"
+		(shape input)
+		(at 96.52 102.87 180)
+		(effects
+			(font
+				(size 1.27 1.27)
+			)
+			(justify right)
+		)
+	)
+	(hierarchical_label "DRDY"
+		(shape input)
+		(at 96.52 92.71 180)
+		(effects
+			(font
+				(size 1.27 1.27)
+			)
+			(justify right)
+		)
+	)
+	(hierarchical_label "CS"
+		(shape input)
+		(at 96.52 100.33 180)
+		(effects
+			(font
+				(size 1.27 1.27)
+			)
+			(justify right)
+		)
+	)
+	(hierarchical_label "SCLK"
+		(shape input)
+		(at 96.52 97.79 180)
+		(effects
+			(font
+				(size 1.27 1.27)
+			)
+			(justify right)
 		)
 	)
@@
 		(on_board yes)
 		(dnp no)
-		(property "Reference" "U?"
+		(property "Reference" "U9"
 			(at 112.014 106.934 0)
 			(effects
@@
 			(project "MCU"
 				(path "/56b3f3ef-07ec-480e-b5f8-5a7fd51b01f6/6dd66391-ee5e-4fdd-bdf7-d4accfe8248c"
-					(reference "U?")
+					(reference "U9")
 					(unit 1)
 				)

Commit message: final changes
Parts:
- C28, C29: footprint Capacitor_SMD:C_0201_0603Metric_Pad0.64x0.40mm_HandSolder -> Capacitor_SMD:C_0603_1608Metric_Pad1.08x0.95mm_HandSolder
- R15, R16, R17, R18: footprint Resistor_SMD:R_0201_0603Metric_Pad0.64x0.40mm_HandSolder -> Resistor_SMD:R_0603_1608Metric_Pad0.98x0.95mm_HandSolder
Changed lines of the file:
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@@
 			)
 		)
-		(property "Footprint" "Resistor_SMD:R_0201_0603Metric_Pad0.64x0.40mm_HandSolder"
+		(property "Footprint" "Resistor_SMD:R_0603_1608Metric_Pad0.98x0.95mm_HandSolder"
 			(at 140.97 119.888 90)
 			(effects
@@
 			)
 		)
-		(property "Footprint" "Resistor_SMD:R_0201_0603Metric_Pad0.64x0.40mm_HandSolder"
+		(property "Footprint" "Resistor_SMD:R_0603_1608Metric_Pad0.98x0.95mm_HandSolder"
 			(at 140.97 104.648 90)
 			(effects
@@
 			)
 		)
-		(property "Footprint" "Capacitor_SMD:C_0201_0603Metric_Pad0.64x0.40mm_HandSolder"
+		(property "Footprint" "Capacitor_SMD:C_0603_1608Metric_Pad1.08x0.95mm_HandSolder"
 			(at 106.9848 74.93 0)
 			(effects
@@
 			)
 		)
-		(property "Datasheet" "https://search.murata.co.jp/Ceramy/image/img/A01X/G101/ENG/GRM033C71C104KE14-01.pdf"
+		(property "Datasheet" "https://www.mouser.com/datasheet/3/72/1/KEM_C1002_X7R_SMD.pdf"
 			(at 107.95 78.74 0)
 			(effects
@@
 			)
 		)
-		(property "Description" "CAP CER 0.1UF 16V X7S 0201"
+		(property "Description" "Multilayer Ceramic Capacitors MLCC - SMD/SMT 50V 0.1uF X7R 0603 10%"
 			(at 107.95 78.74 0)
 			(effects
@@
 			)
 		)
-		(property "Footprint" "Resistor_SMD:R_0201_0603Metric_Pad0.64x0.40mm_HandSolder"
+		(property "Footprint" "Resistor_SMD:R_0603_1608Metric_Pad0.98x0.95mm_HandSolder"
 			(at 140.97 110.998 90)
 			(effects
@@
 			)
 		)
-		(property "Footprint" "Resistor_SMD:R_0201_0603Metric_Pad0.64x0.40mm_HandSolder"
+		(property "Footprint" "Resistor_SMD:R_0603_1608Metric_Pad0.98x0.95mm_HandSolder"
 			(at 140.97 122.428 90)
 			(effects
@@
 			)
 		)
-		(property "Footprint" "Capacitor_SMD:C_0201_0603Metric_Pad0.64x0.40mm_HandSolder"
+		(property "Footprint" "Capacitor_SMD:C_0603_1608Metric_Pad1.08x0.95mm_HandSolder"
 			(at 121.6152 82.55 0)
 			(effects
@@
 			)
 		)
-		(property "Datasheet" "https://search.murata.co.jp/Ceramy/image/img/A01X/G101/ENG/GRM033C71C104KE14-01.pdf"
+		(property "Datasheet" "https://www.mouser.com/datasheet/3/72/1/KEM_C1002_X7R_SMD.pdf"
 			(at 120.65 78.74 0)
 			(effects
@@
 			)
 		)
-		(property "Description" "CAP CER 0.1UF 16V X7S 0201"
+		(property "Description" "Multilayer Ceramic Capacitors MLCC - SMD/SMT 50V 0.1uF X7R 0603 10%"
 			(at 120.65 78.74 0)
 			(effects
