File: RTD/RTD.kicad_sch (KiCad schematic)
At the start: 11 parts, among them J1 Conn_01x04, U1 MAX31865xAP, U2 Nucleo_L432KC

Commit message: Cleaned up traces in MCU layout
Parts:
- U2: footprint UTSVT Special:NucleoL432KC -> UTSVT STM32:NucleoL432KC
Connections:
- net PA7: now reaches U2.25 (A6)
- net PA7: now also U1.14 (SDI)
- net D11: no longer names the net of U2.14 (D11)
- net D11: no longer U1.14 (SDI)
- net D12 renamed PA6
- net D13 renamed PA5
- net PA4: no longer names the net of U2.22 (A3)
- net PA4: no longer U1.16 (~{CS})
- new net D3: U1.16 (~{CS})
- no-connect marks 23 -> 24
Other:
- note added: "MAX31865 CS → MCU SSEL (or GPIO used as CS)- D3 SPI1(PA4 SPI3_SSEL) MAX31865 SCLK → MCU SCLK - PA5 SPI1(D13 SPI3_SCLK) MAX31865 SDI → MCU MOSI - PA7 SPI1(D11 SPI3_MOSI) MAX31865 SDO → MCU MISO - PA6 SPI1(D12 SPI3_MISO) MAX31865 DRDY → digital input pin (HIGH when MAX is busy performing conversion. LOW when new measurement is ready)- D7 Not enough pins on the Current Regulating MCU. Will use anoth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"
- note removed: "MAX31865 CS → MCU SSEL (or GPIO used as CS)- PA4 SPI3_SSEL MAX31865 SCLK → MCU SCLK - D13 SPI3_SCLK MAX31865 SDI → MCU MOSI - D11 SPI3_MOSI MAX31865 SDO → MCU MISO - D12 SPI3_MISO MAX31865 DRDY → digital input pin (HIGH when MAX is busy performing conversion. LOW when new measurement is ready)- D7 Not enough pins on the Current Regulating MCU. Will use another one."
Changed lines of the file:
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@@
 		)
 	)
-	(text "MAX31865 CS  →  MCU SSEL (or GPIO used as CS)- PA4 SPI3_SSEL\nMAX31865 SCLK → MCU SCLK - D13 SPI3_SCLK\nMAX31865 SDI  → MCU MOSI - D11 SPI3_MOSI\nMAX31865 SDO  → MCU MISO - D12 SPI3_MISO\nMAX31865 DRDY → digital input pin (HIGH when MAX is busy\n			performing conversion. LOW when new\n			measurement is ready)- D7\n\nNot enough pins on the Current Regulating MCU. Will use another one."
+	(text "MAX31865 CS  →  MCU SSEL (or GPIO used as CS)- D3 SPI1(PA4 SPI3_SSEL)\nMAX31865 SCLK → MCU SCLK - PA5 SPI1(D13 SPI3_SCLK)\nMAX31865 SDI  → MCU MOSI - PA7 SPI1(D11 SPI3_MOSI)\nMAX31865 SDO  → MCU MISO - PA6 SPI1(D12 SPI3_MISO)\nMAX31865 DRDY → digital input pin (HIGH when MAX is busy\n			performing conversion. LOW when new\n			measurement is ready)- D7\n\nNot enough pins on the Current Regulating MCU. Will use another one."
 		(exclude_from_sim no)
 		(at 60.452 35.814 0)
@@
 	)
 	(no_connect
+		(at 77.47 105.41)
+	)
+	(no_connect
+		(at 102.87 82.55)
+	)
+	(no_connect
+		(at 77.47 100.33)
+	)
+	(no_connect
+		(at 77.47 85.09)
+	)
+	(no_connect
+		(at 77.47 97.79)
+	)
+	(no_connect
+		(at 77.47 80.01)
+	)
+	(no_connect
+		(at 102.87 72.39)
+	)
+	(no_connect
+		(at 102.87 77.47)
+	)
+	(no_connect
+		(at 102.87 100.33)
+	)
+	(no_connect
+		(at 102.87 92.71)
+	)
+	(no_connect
+		(at 102.87 87.63)
+	)
+	(no_connect
+		(at 102.87 80.01)
+	)
+	(no_connect
+		(at 102.87 90.17)
+	)
+	(no_connect
+		(at 102.87 97.79)
+	)
+	(no_connect
+		(at 77.47 72.39)
+	)
+	(no_connect
+		(at 77.47 90.17)
+	)
+	(no_connect
+		(at 77.47 92.71)
+	)
+	(no_connect
 		(at 102.87 95.25)
 	)
-	(no_connect
-		(at 102.87 82.55)
-	)
-	(no_connect
-		(at 77.47 100.33)
-	)
-	(no_connect
-		(at 77.47 85.09)
-	)
-	(no_connect
-		(at 77.47 97.79)
-	)
-	(no_connect
-		(at 77.47 80.01)
-	)
-	(no_connect
-		(at 102.87 72.39)
-	)
-	(no_connect
-		(at 102.87 77.47)
-	)
-	(no_connect
-		(at 102.87 100.33)
-	)
-	(no_connect
-		(at 102.87 87.63)
-	)
-	(no_connect
-		(at 102.87 80.01)
-	)
-	(no_connect
-		(at 102.87 90.17)
-	)
-	(no_connect
-		(at 102.87 97.79)
-	)
-	(no_connect
-		(at 102.87 85.09)
-	)
-	(no_connect
-		(at 77.47 72.39)
-	)
-	(no_connect
-		(at 77.47 90.17)
-	)
-	(no_connect
-		(at 77.47 92.71)
-	)
 	(wire
 		(pts
@@
 	(wire
 		(pts
-			(xy 102.87 92.71) (xy 104.14 92.71)
-		)
-		(stroke
-			(width 0)
-			(type default)
-		)
-	)
-	(wire
-		(pts
 			(xy 76.2 107.95) (xy 77.47 107.95)
 		)
@@
 	(wire
 		(pts
-			(xy 76.2 105.41) (xy 77.47 105.41)
-		)
-		(stroke
-			(width 0)
-			(type default)
-		)
-	)
-	(wire
-		(pts
 			(xy 127 78.74) (xy 128.27 78.74)
 		)
@@
 	(wire
 		(pts
+			(xy 104.14 85.09) (xy 102.87 85.09)
+		)
+		(stroke
+			(width 0)
+			(type default)
+		)
+	)
+	(wire
+		(pts
 			(xy 165.1 104.14) (xy 166.37 104.14)
 		)
@@
 		)
 	)
-	(label "D13"
+	(label "PA5"
 		(at 127 83.82 180)
 		(effects
@@
 		)
 	)
-	(label "PA4"
-		(at 104.14 92.71 0)
-		(effects
-			(font
-				(size 1.27 1.27)
-			)
-			(justify left bottom)
-		)
-	)
-	(label "D12"
+	(label "PA6"
 		(at 76.2 107.95 180)
-		(effects
-			(font
-				(size 1.27 1.27)
-			)
-			(justify right bottom)
-		)
-	)
-	(label "D11"
-		(at 76.2 105.41 180)
 		(effects
 			(font
@@
 		)
 	)
-	(label "D12"
+	(label "PA6"
 		(at 127 88.9 180)
 		(effects
@@
 		)
 	)
-	(label "D13"
+	(label "PA5"
 		(at 104.14 107.95 0)
 		(effects
@@
 		)
 	)
-	(label "D11"
+	(label "PA7"
 		(at 127 81.28 180)
 		(effects
@@
 		)
 	)
-	(label "PA4"
+	(label "D3"
 		(at 127 86.36 180)
 		(effects
@@
 			)
 			(justify right bottom)
+		)
+	)
+	(label "PA7"
+		(at 104.14 85.09 0)
+		(effects
+			(font
+				(size 1.27 1.27)
+			)
+			(justify left bottom)
 		)
 	)
@@
 			)
 		)
-		(property "Footprint" "UTSVT Special:NucleoL432KC"
+		(property "Footprint" "UTSVT STM32:NucleoL432KC"
 			(at 90.17 97.79 0)
 			(effects
